Commit message: Bump to ROS2 Jazzy
This bumps the project to ROS2 Jazzy[1], based on Ubuntu Noble 24.04
LTS[2].

Fixes:

	In file included from /home/gportay/src/abmi-software/Robot5A-Simulation/src/robot_control/src/moveit_control_simple.cpp:5:
	/opt/ros/jazzy/include/moveit_ros_planning_interface/moveit/move_group_interface/move_group_interface.h:51:77: note: ‘#pragma message: .h header is obsolete. Please use the .hpp header instead.’
	   51 | #pragma message(".h header is obsolete. Please use the .hpp header instead.")
	      |                                                                             ^

And fixes:

	/home/gportay/src/abmi-software/Robot5A-Simulation/src/robot_control/src/aruco_detector_single.cpp:5:10: fatal error: cv_bridge/cv_bridge.h: No such file or directory
	    5 | #include <cv_bridge/cv_bridge.h>
	      |          ^~~~~~~~~~~~~~~~~~~~~~~
	compilation terminated.

TODO: Fix the ArUco Markers[5].

[1]: https://docs.ros.org/en/jazzy/index.html
[2]: https://ubuntu.com/blog/tag/ubuntu-24-04-lts
[3]: https://gazebosim.org/docs/latest/migrating_gazebo_classic_ros2_packages/
[4]: https://gazebosim.org/api/sim/8/migrationsdf.html
[5]: https://gazebosim.org/api/sim/8/migrationsdf.html#:~:text=Materials

File: src/robot_description/urdf/aruco.urdf.xacro (robot description, xacro)
@@ -32,5 +32,6 @@
     <!-- Assign custom material to the plane -->
     <gazebo reference="aruco_plane_${plane_number}">
-      <material>id${plane_number}_Plane_Material</material>
+      <!-- FIXME -->
+      <material>Gazebo/Red</material>
       <disable_collision>true</disable_collision>
     </gazebo>

File: src/robot_description/urdf/r5a_v_ros.urdf.xacro (robot description, xacro)
@@ -724,5 +724,5 @@
   <ros2_control name="GazeboSystem" type="system">
     <hardware>
-      <plugin>gazebo_ros2_control/GazeboSystem</plugin>
+      <plugin>gz_ros2_control/GazeboSimSystem</plugin>
       <param name="use_sim_time" type="bool">true</param>
     </hardware>
@@ -806,29 +806,12 @@
   </ros2_control>
   <gazebo>
-    <plugin name="gazebo_ros2_control" filename="libgazebo_ros2_control.so">
+    <plugin name="gz_ros2_control::GazeboSimROS2ControlPlugin" filename="libgz_ros2_control-system.so">
     <robotNamespace>/</robotNamespace>
       <robot_param>robot_description</robot_param>
       <robot_param_node>robot_state_publisher</robot_param_node>
-      <robot_sim_type>gazebo_ros2_control/GazeboSystem</robot_sim_type>
+      <robot_sim_type>gz_ros2_control/GazeboSystem</robot_sim_type>
       <parameters>$(find robot_description)/config/controller.yaml</parameters>
       <controller_manager_name>controller_manager</controller_manager_name>
       <use_sim_time>true</use_sim_time>
-    </plugin>
-  </gazebo>
-  <gazebo>
-    <plugin name="gazebo_ros_joint_pose_trajectory" filename="libgazebo_ros_joint_pose_trajectory.so">
-        <update_rate>50
-        </update_rate>
-        <joint_name>R0_Yaw</joint_name>
-        <joint_name>R1_Pitch</joint_name>
-        <joint_name>R2_Pitch</joint_name>
-        <joint_name>R3_Yaw</joint_name>
-        <joint_name>R4_Pitch</joint_name>
-        <joint_name>ServoGear</joint_name>
-        <joint_name>LeftGripper</joint_name>
-        <joint_name>LeftPivotArm</joint_name>
-        <joint_name>PassifGear</joint_name>
-        <joint_name>RightGripper</joint_name>
-        <joint_name>RightPivotArm</joint_name>
     </plugin>
   </gazebo>
@@ -876,19 +859,9 @@
           <stddev>0.007</stddev>
         </noise>
+        <camera_info_topic>camera_info</camera_info_topic>
       </camera>
-      <plugin name="camera_controller1" filename="libgazebo_ros_camera.so">
-        <alwaysOn>true</alwaysOn>
-        <updateRate>0.0</updateRate>
-        <cameraName>mybot/camera1</cameraName>
-        <imageTopicName>image_raw</imageTopicName>
-        <cameraInfoTopicName>camera_info</cameraInfoTopicName>
-        <frameName>camera_link1</frameName>
-        <hackBaseline>0.07</hackBaseline>
-        <distortionK1>0.0</distortionK1>
-        <distortionK2>0.0</distortionK2>
-        <distortionK3>0.0</distortionK3>
-        <distortionT1>0.0</distortionT1>
-        <distortionT2>0.0</distortionT2>
-      </plugin>
+      <always_on>true</always_on>
+      <topic>camera/image_raw</topic>
+      <gz_frame_id>camera_link1</gz_frame_id>
     </sensor>
   </gazebo>
@@ -936,19 +909,10 @@
           <stddev>0.007</stddev>
         </noise>
+        <camera_info_topic>camera_info2</camera_info_topic>
       </camera>
-      <plugin name="camera_controller2" filename="libgazebo_ros_camera.so">
-        <alwaysOn>true</alwaysOn>
-        <updateRate>0.0</updateRate>
-        <cameraName>mybot/camera2</cameraName>
-        <imageTopicName>image_raw2</imageTopicName>
-        <cameraInfoTopicName>camera_info2</cameraInfoTopicName>
-        <frameName>camera_link2</frameName>
-        <hackBaseline>0.07</hackBaseline>
-        <distortionK1>0.0</distortionK1>
-        <distortionK2>0.0</distortionK2>
-        <distortionK3>0.0</distortionK3>
-        <distortionT1>0.0</distortionT1>
-        <distortionT2>0.0</distortionT2>
-      </plugin>
+      <always_on>true</always_on>
+      <visualize>true</visualize>
+      <gz_frame_id>camera_link2</gz_frame_id>
+      <topic>camera/image_raw</topic>
     </sensor>
   </gazebo>
