Commit message: Add files via upload

File: src/robot_description/urdf/r5a_v_ros.urdf.xacro (robot description, xacro)
@@ -105,4 +105,5 @@
       effort="5"
       velocity="1" />
+    <hardwareInterface>position</hardwareInterface>
   </joint>
   <link
@@ -163,4 +164,5 @@
       effort="5"
       velocity="1" />
+    <hardwareInterface>position</hardwareInterface>
   </joint>
   <link
@@ -221,4 +223,5 @@
       effort="5"
       velocity="1" />
+    <hardwareInterface>position</hardwareInterface>
   </joint>
   <link
@@ -279,4 +282,5 @@
       effort="5"
       velocity="1" />
+    <hardwareInterface>position</hardwareInterface>
   </joint>
   <link
@@ -337,4 +341,5 @@
       effort="5"
       velocity="1" />
+    <hardwareInterface>position</hardwareInterface>
   </joint>
   <link
@@ -395,4 +400,5 @@
       effort="5"
       velocity="1" />
+    <hardwareInterface>position</hardwareInterface>
   </joint>
   <link
@@ -453,4 +459,5 @@
       effort="5"
       velocity="1" />
+   <hardwareInterface>position</hardwareInterface>
   </joint>
   <link
@@ -511,4 +518,5 @@
       effort="5"
       velocity="1" />
+    <hardwareInterface>position</hardwareInterface>
   </joint>
   <link
@@ -569,4 +577,5 @@
       effort="5"
       velocity="1" />
+    <hardwareInterface>position</hardwareInterface>
   </joint>
   <link
@@ -627,4 +636,5 @@
       effort="5"
       velocity="1" />
+    <hardwareInterface>position</hardwareInterface>
   </joint>
   <link
@@ -685,135 +695,108 @@
       effort="5"
       velocity="1" />
-  </joint>
-  <gazebo reference="base_link">
-    <material>Gazebo/White</material>
-  </gazebo>
-  <gazebo reference="R5A_link1">
-    <material>Gazebo/White</material>
-  </gazebo>
-  <gazebo reference="R5A_link2">
-    <material>Gazebo/White</material>
-  </gazebo>
-  <gazebo reference="R5A_link3">
-    <material>Gazebo/White</material>
-  </gazebo>
-  <gazebo reference="R5A_link4">
-    <material>Gazebo/White</material>
-  </gazebo>
-  <gazebo reference="R5A_link5">
-    <material>Gazebo/Black</material>
-  </gazebo>
-  <gazebo reference="R5A_GripperRight_Link1">
-    <material>Gazebo/White</material>
-  </gazebo>
-  <gazebo reference="R5A_GripperRight_Link2">
-    <material>Gazebo/Black</material>
-  </gazebo>
-  <gazebo reference="R5A_GripperRight_Link3">
-    <material>Gazebo/White</material>
-  </gazebo>
-  <gazebo reference="R5A_GripperLeft_Link1">
-    <material>Gazebo/White</material>
-  </gazebo>
-  <gazebo reference="R5A_GripperLeft_Link2">
-    <material>Gazebo/Black</material>
-  </gazebo>
-  <gazebo reference="R5A_GripperLeft_Link3">
-    <material>Gazebo/White</material>
-  </gazebo>
-  <ros2_control name="GazeboSystem" type="system">
-    <hardware>
-      <plugin>gz_ros2_control/GazeboSimSystem</plugin>
-      <param name="use_sim_time" type="bool">true</param>
-    </hardware>
+    <hardwareInterface>position</hardwareInterface>
+  </joint>
+<!-- Automatically updated r5a_v_ros.urdf.xacro with <transmission> blocks -->
+<!-- You still need to insert this into your full file manually at the correct spot -->
+<!-- Begin transmission blocks -->
+  <transmission name="R0_Yaw_trans">
+    <type>transmission_interface/SimpleTransmission</type>
     <joint name="R0_Yaw">
-      <command_interface name="position"/>
-      <state_interface name="position">
-        <param name="initial_value">0.0</param>
-      </state_interface>
-      <state_interface name="velocity"/>
-    </joint>
+      <hardwareInterface>hardware_interface/PositionJointInterface</hardwareInterface>
+    </joint>
+    <actuator name="R0_Yaw_motor">
+      <hardwareInterface>hardware_interface/PositionJointInterface</hardwareInterface>
+    </actuator>
+  </transmission>
+  <transmission name="R1_Pitch_trans">
+    <type>transmission_interface/SimpleTransmission</type>
     <joint name="R1_Pitch">
-      <command_interface name="position"/>
-      <state_interface name="position">
-        <param name="initial_value">0.0</param>
-      </state_interface>
-      <state_interface name="velocity"/>
-    </joint>
+      <hardwareInterface>hardware_interface/PositionJointInterface</hardwareInterface>
+    </joint>
+    <actuator name="R1_Pitch_motor">
+      <hardwareInterface>hardware_interface/PositionJointInterface</hardwareInterface>
+    </actuator>
+  </transmission>
+  <transmission name="R2_Pitch_trans">
+    <type>transmission_interface/SimpleTransmission</type>
     <joint name="R2_Pitch">
-      <command_interface name="position"/>
-      <state_interface name="position">
-        <param name="initial_value">0.0</param>
-      </state_interface>
-      <state_interface name="velocity"/>
-    </joint>
+      <hardwareInterface>hardware_interface/PositionJointInterface</hardwareInterface>
+    </joint>
+    <actuator name="R2_Pitch_motor">
+      <hardwareInterface>hardware_interface/PositionJointInterface</hardwareInterface>
+    </actuator>
+  </transmission>
+  <transmission name="R3_Yaw_trans">
+    <type>transmission_interface/SimpleTransmission</type>
     <joint name="R3_Yaw">
-      <command_interface name="position"/>
-      <state_interface name="position">
-        <param name="initial_value">0.0</param>
-      </state_interface>
-      <state_interface name="velocity"/>
-    </joint>
+      <hardwareInterface>hardware_interface/PositionJointInterface</hardwareInterface>
+    </joint>
+    <actuator name="R3_Yaw_motor">
+      <hardwareInterface>hardware_interface/PositionJointInterface</hardwareInterface>
+    </actuator>
+  </transmission>
+  <transmission name="R4_Pitch_trans">
+    <type>transmission_interface/SimpleTransmission</type>
     <joint name="R4_Pitch">
-      <command_interface name="position"/>
-      <state_interface name="position">
-        <param name="initial_value">0.0</param>
-      </state_interface>
-      <state_interface name="velocity"/>
-    </joint>
+      <hardwareInterface>hardware_interface/PositionJointInterface</hardwareInterface>
+    </joint>
+    <actuator name="R4_Pitch_motor">
+      <hardwareInterface>hardware_interface/PositionJointInterface</hardwareInterface>
+    </actuator>
+  </transmission>
+  <transmission name="ServoGear_trans">
+    <type>transmission_interface/SimpleTransmission</type>
     <joint name="ServoGear">
-      <command_interface name="position"/>
-      <state_interface name="position">
-        <param name="initial_value">0.0</param>
-      </state_interface>
-      <state_interface name="velocity"/>
-    </joint>
+      <hardwareInterface>hardware_interface/PositionJointInterface</hardwareInterface>
+    </joint>
+    <actuator name="ServoGear_motor">
+      <hardwareInterface>hardware_interface/PositionJointInterface</hardwareInterface>
+    </actuator>
+  </transmission>
+  <transmission name="LeftGripper_trans">
+    <type>transmission_interface/SimpleTransmission</type>
     <joint name="LeftGripper">
-      <command_interface name="position"/>
-      <state_interface name="position">
-        <param name="initial_value">0.0</param>
-      </state_interface>
-      <state_interface name="velocity"/>
-    </joint>
+      <hardwareInterface>hardware_interface/PositionJointInterface</hardwareInterface>
+    </joint>
+    <actuator name="LeftGripper_motor">
+      <hardwareInterface>hardware_interface/PositionJointInterface</hardwareInterface>
+    </actuator>
+  </transmission>
+  <transmission name="LeftPivotArm_trans">
+    <type>transmission_interface/SimpleTransmission</type>
     <joint name="LeftPivotArm">
-      <command_interface name="position"/>
-      <state_interface name="position">
-        <param name="initial_value">0.0</param>
-      </state_interface>
-      <state_interface name="velocity"/>
-    </joint>
+      <hardwareInterface>hardware_interface/PositionJointInterface</hardwareInterface>
+    </joint>
+    <actuator name="LeftPivotArm_motor">
+      <hardwareInterface>hardware_interface/PositionJointInterface</hardwareInterface>
+    </actuator>
+  </transmission>
+  <transmission name="PassifGear_trans">
+    <type>transmission_interface/SimpleTransmission</type>
     <joint name="PassifGear">
-      <command_interface name="position"/>
-      <state_interface name="position">
-        <param name="initial_value">0.0</param>
-      </state_interface>
-      <state_interface name="velocity"/>
-    </joint>
+      <hardwareInterface>hardware_interface/PositionJointInterface</hardwareInterface>
+    </joint>
+    <actuator name="PassifGear_motor">
+      <hardwareInterface>hardware_interface/PositionJointInterface</hardwareInterface>
+    </actuator>
+  </transmission>
+  <transmission name="RightGripper_trans">
+    <type>transmission_interface/SimpleTransmission</type>
     <joint name="RightGripper">
-      <command_interface name="position"/>
-      <state_interface name="position">
-        <param name="initial_value">0.0</param>
-      </state_interface>
-      <state_interface name="velocity"/>
-    </joint>
+      <hardwareInterface>hardware_interface/PositionJointInterface</hardwareInterface>
+    </joint>
+    <actuator name="RightGripper_motor">
+      <hardwareInterface>hardware_interface/PositionJointInterface</hardwareInterface>
+    </actuator>
+  </transmission>
+  <transmission name="RightPivotArm_trans">
+    <type>transmission_interface/SimpleTransmission</type>
     <joint name="RightPivotArm">
-      <command_interface name="position"/>
-      <state_interface name="position">
-        <param name="initial_value">0.0</param>
-      </state_interface>
-      <state_interface name="velocity"/>
-    </joint>
-  </ros2_control>
-  <gazebo>
-    <plugin name="gz_ros2_control::GazeboSimROS2ControlPlugin" filename="libgz_ros2_control-system.so">
-    <robotNamespace>/</robotNamespace>
-      <robot_param>robot_description</robot_param>
-      <robot_param_node>robot_state_publisher</robot_param_node>
-      <robot_sim_type>gz_ros2_control/GazeboSystem</robot_sim_type>
-      <parameters>$(find robot_description)/config/controller.yaml</parameters>
-      <controller_manager_name>controller_manager</controller_manager_name>
-      <use_sim_time>true</use_sim_time>
-    </plugin>
-  </gazebo>
+      <hardwareInterface>hardware_interface/PositionJointInterface</hardwareInterface>
+    </joint>
+    <actuator name="RightPivotArm_motor">
+      <hardwareInterface>hardware_interface/PositionJointInterface</hardwareInterface>
+    </actuator>
+  </transmission>
 <!-- First Camera -->
   <link name="camera_link1">
@@ -831,7 +814,4 @@
     </collision>
   </link>
-  <gazebo reference="camera_link1">
-    <material>Gazebo/Black</material>
-  </gazebo>
   <joint name="camera_joint1" type="fixed">
     <origin xyz="1.2 0.0 0.45" rpy="0 0 3.14159"/>
@@ -840,30 +820,4 @@
   </joint>
   <!-- Gazebo Camera Plugin for First Camera -->
-  <gazebo reference="camera_link1">
-    <sensor type="camera" name="camera1">
-      <update_rate>30.0</update_rate>
-      <camera name="head1">
-        <horizontal_fov>1.3962634</horizontal_fov>
-        <image>
-          <width>1920</width>
-          <height>1080</height>
-          <format>R8G8B8</format>
-        </image>
-        <clip>
-          <near>0.02</near>
-          <far>300</far>
-        </clip>
-        <noise>
-          <type>gaussian</type>
-          <mean>0.0</mean>
-          <stddev>0.007</stddev>
-        </noise>
-        <camera_info_topic>camera_info</camera_info_topic>
-      </camera>
-      <always_on>true</always_on>
-      <topic>camera/image_raw</topic>
-      <gz_frame_id>camera_link1</gz_frame_id>
-    </sensor>
-  </gazebo>
   <!-- Second Camera -->
   <link name="camera_link2">
@@ -881,7 +835,4 @@
     </collision>
   </link>
-  <gazebo reference="camera_link2">
-    <material>Gazebo/Black</material>
-  </gazebo>
   <joint name="camera_joint2" type="fixed">
     <origin xyz="-0.5 0.5 1" rpy="0 0.7854 -0.7854"/> <!-- Adjust xyz to place in front of the first camera -->
@@ -889,31 +840,183 @@
     <child link="camera_link2"/>
   </joint>
-  <!-- Gazebo Camera Plugin for Second Camera -->
-  <gazebo reference="camera_link2">
-    <sensor type="camera" name="camera2">
-      <update_rate>30.0</update_rate>
-      <camera name="head2">
-        <horizontal_fov>1.3962634</horizontal_fov>
-        <image>
-          <width>1920</width>
-          <height>1080</height>
-          <format>R8G8B8</format>
-        </image>
-        <clip>
-          <near>0.02</near>
-          <far>300</far>
-        </clip>
-        <noise>
-          <type>gaussian</type>
-          <mean>0.0</mean>
-          <stddev>0.007</stddev>
-        </noise>
-        <camera_info_topic>camera_info2</camera_info_topic>
-      </camera>
-      <always_on>true</always_on>
-      <visualize>true</visualize>
-      <gz_frame_id>camera_link2</gz_frame_id>
-      <topic>camera/image_raw</topic>
-    </sensor>
+  <!-- Gazebo  -->
+<!-- Add this for Gazebo ros2_control plugin integration -->
+  <gazebo>
+    <plugin name="gz_ros2_control::GazeboSimROS2ControlPlugin" filename="libgz_ros2_control-system.so">
+      <ros2_control>
+        <robot_param>robot_description</robot_param>
+        <parameters>/home/rothvichea/ros2_jazzy/install/robot_control/share/robot_control/config/controller.yaml</parameters>
+      </ros2_control>
+    </plugin>
   </gazebo>
+  <transmission name="R0_Yaw_trans">
+    <type>transmission_interface/SimpleTransmission</type>
+    <joint name="R0_Yaw">
+      <hardwareInterface>position</hardwareInterface>
+    </joint>
+    <actuator name="R0_Yaw_motor">
+      <hardwareInterface>position</hardwareInterface>
+      <mechanicalReduction>1</mechanicalReduction>
+    </actuator>
+  </transmission>
+  <transmission name="R1_Pitch_trans">
+    <type>transmission_interface/SimpleTransmission</type>
+    <joint name="R1_Pitch">
+      <hardwareInterface>position</hardwareInterface>
+    </joint>
+    <actuator name="R1_Pitch_motor">
+      <hardwareInterface>position</hardwareInterface>
+      <mechanicalReduction>1</mechanicalReduction>
+    </actuator>
+  </transmission>
+  <transmission name="R2_Pitch_trans">
+    <type>transmission_interface/SimpleTransmission</type>
+    <joint name="R2_Pitch">
+      <hardwareInterface>position</hardwareInterface>
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
Commit message: Remplacer le contenu de la branche distante

File: src/robot_description/urdf/r5a_v_ros.urdf.xacro (robot description, xacro)
@@ -1,5 +1,5 @@
 <?xml version="1.0" encoding="utf-8"?>
 <robot name="armr5" xmlns:xacro="http://www.ros.org/wiki/xacro">
-  <xacro:include filename="aruco.urdf.xacro" />
+  <!-- <xacro:include filename="aruco.urdf.xacro" /> -->
   <link name="world"></link>
   <joint name="base_joint" type="fixed">
@@ -686,39 +686,68 @@
       velocity="1" />
   </joint>
+  <!-- MATÉRIAUX PLASTIQUE NOIR MAT PERSONNALISÉS -->
+  <!-- Corps principal du robot en plastique noir mat -->
   <gazebo reference="base_link">
-    <material>Gazebo/White</material>
+    <material>PlasticBlackGlossy</material>
+    <mu1>0.8</mu1>
+    <mu2>0.8</mu2>
+    <kp>1000000.0</kp>
+    <kd>1.0</kd>
   </gazebo>
   <gazebo reference="R5A_link1">
-    <material>Gazebo/White</material>
+    <material>PlasticBlackGlossy</material>
+    <mu1>0.8</mu1>
+    <mu2>0.8</mu2>
   </gazebo>
   <gazebo reference="R5A_link2">
-    <material>Gazebo/White</material>
+    <material>PlasticBlackGlossy</material>
+    <mu1>0.8</mu1>
+    <mu2>0.8</mu2>
   </gazebo>
   <gazebo reference="R5A_link3">
-    <material>Gazebo/White</material>
+    <material>PlasticBlackGlossy</material>
+    <mu1>0.8</mu1>
+    <mu2>0.8</mu2>
   </gazebo>
   <gazebo reference="R5A_link4">
-    <material>Gazebo/White</material>
+    <material>PlasticBlackGlossy</material>
+    <mu1>0.8</mu1>
+    <mu2>0.8</mu2>
   </gazebo>
   <gazebo reference="R5A_link5">
-    <material>Gazebo/Black</material>
-  </gazebo>
+    <material>PlasticBlackGlossy</material>
+    <mu1>0.8</mu1>
+    <mu2>0.8</mu2>
+  </gazebo>
+  <!-- Gripper en plastique noir légèrement brillant pour contraste -->
   <gazebo reference="R5A_GripperRight_Link1">
-    <material>Gazebo/White</material>
+    <material>PlasticBlackGlossy</material>
+    <mu1>0.9</mu1>
+    <mu2>0.9</mu2>
   </gazebo>
   <gazebo reference="R5A_GripperRight_Link2">
-    <material>Gazebo/Black</material>
+    <material>PlasticBlackGlossy</material>
+    <mu1>0.9</mu1>
+    <mu2>0.9</mu2>
   </gazebo>
   <gazebo reference="R5A_GripperRight_Link3">
-    <material>Gazebo/White</material>
+    <material>PlasticOffWhite</material>
+    <mu1>0.9</mu1>
+    <mu2>0.9</mu2>
   </gazebo>
   <gazebo reference="R5A_GripperLeft_Link1">
-    <material>Gazebo/White</material>
+    <material>PlasticBlackGlossy</material>
+    <mu1>0.9</mu1>
+    <mu2>0.9</mu2>
   </gazebo>
   <gazebo reference="R5A_GripperLeft_Link2">
-    <material>Gazebo/Black</material>
+    <material>PlasticBlackGlossy</material>
+    <mu1>0.9</mu1>
+    <mu2>0.9</mu2>
   </gazebo>
   <gazebo reference="R5A_GripperLeft_Link3">
-    <material>Gazebo/White</material>
+    <material>PlasticOffWhite</material>
+    <mu1>0.9</mu1>
+    <mu2>0.9</mu2>
   </gazebo>
   <ros2_control name="GazeboSystem" type="system">
