Commit message: Update r5a_v_ros.urdf.xacro

File: src/robot_description/urdf/r5a_v_ros.urdf.xacro (robot description, xacro)
@@ -1,6 +1,6 @@
-<?xml version="1.0" encoding="utf-8"?>
+<?xml version="1.0"?>
 <robot name="armr5" xmlns:xacro="http://www.ros.org/wiki/xacro">
-  <xacro:include filename="aruco.urdf.xacro" />
-  <link name="world"></link>
+  <!-- Base to world fixed joint -->
+  <link name="world"/>
   <joint name="base_joint" type="fixed">
     <origin xyz="0 0 0" rpy="0 0 0"/>
@@ -8,1014 +8,470 @@
     <child link="base_link"/>
   </joint>
-  <link
-    name="base_link">
-    <inertial>
-      <origin
-        xyz="0.00683000289839214 0.0492858185856111 0.102410796188668"
-        rpy="0 0 0" />
-      <mass
-        value="1.54608760930939" />
+  <!-- base_link -->
+  <link name="base_link">
+    <visual>
+      <origin xyz="0 0 0" rpy="0 0 0" />
+      <geometry>
+        <mesh filename="package://robot_description/meshes/base_link.STL" scale="1 1 1"/>
+      </geometry>
+    </visual>
+    <collision>
+      <geometry>
+        <mesh filename="package://robot_description/meshes/base_link.STL" scale="1 1 1"/>
+      </geometry>
+    </collision>
+    <inertial>
+      <origin xyz="0.00683000289839214 0.0492858185856111 0.102410796188668" rpy="0 0 0" />
+      <mass value="1.54608760930939" />
       <inertia
-        ixx="0.00335325507409126"
-        ixy="-2.743396733147E-05"
-        ixz="6.86594556642029E-08"
-        iyy="0.00381821146815156"
-        iyz="-1.9423420965472E-06"
-        izz="0.00646111115889031" />
-    </inertial>
-    <visual>
-      <origin
-        xyz="0 0 0"
-        rpy="0 0 0" />
-      <geometry>
-        <mesh
-          filename="file://$(find robot_description)/meshes/base_link.STL" />
-      </geometry>
-      <material
-        name="">
-        <color
-          rgba="0.792156862745098 0.819607843137255 0.933333333333333 1" />
-      </material>
-    </visual>
-    <collision>
-      <origin
-        xyz="0 0 0"
-        rpy="0 0 0" />
-      <geometry>
-        <mesh
-          filename="file://$(find robot_description)/meshes/base_link.STL" />
-      </geometry>
-    </collision>
-  </link>
-  <link
-    name="R5A_link1">
-    <inertial>
-      <origin
-        xyz="-0.000863539879134213 0.0792884229151367 0.000217126309188408"
-        rpy="0 0 0" />
-      <mass
-        value="2.08660345546666" />
-      <inertia
-        ixx="0.00705202984610834"
-        ixy="4.18495769536855E-07"
-        ixz="-5.35090527857546E-08"
-        iyy="0.00650257727022909"
-        iyz="-7.95450001919519E-07"
-        izz="0.00859235014286563" />
-    </inertial>
-    <visual>
-      <origin
-        xyz="0 0 0"
-        rpy="0 0 0" />
-      <geometry>
-        <mesh
-          filename="file://$(find robot_description)/meshes/R5A_link1.STL" />
-      </geometry>
-      <material
-        name="">
-        <color
-          rgba="0.792156862745098 0.819607843137255 0.933333333333333 1" />
-      </material>
-    </visual>
-    <collision>
-      <origin
-        xyz="0 0 0"
-        rpy="0 0 0" />
-      <geometry>
-        <mesh
-          filename="file://$(find robot_description)/meshes/R5A_link1.STL" />
-      </geometry>
-    </collision>
-  </link>
-  <joint
-    name="R0_Yaw"
-    type="revolute">
-    <origin
-      xyz="0.00685726045199512 0 0.15825"
-      rpy="1.5707963267949 0 0" />
-    <parent
-      link="base_link" />
-    <child
-      link="R5A_link1" />
-    <axis
-      xyz="0 1 0" />
-    <limit
-      lower="-1.5"
-      upper="1.5"
-      effort="5"
-      velocity="1" />
-    <hardwareInterface>position</hardwareInterface>
-  </joint>
-  <link
-    name="R5A_link2">
-    <inertial>
-      <origin
-        xyz="0.000590340031700784 0.0792749789345383 -1.60575865215828E-05"
-        rpy="0 0 0" />
-      <mass
-        value="1.92247082198063" />
-      <inertia
-        ixx="0.00487699383852877"
-        ixy="-3.67976990627086E-05"
-        ixz="1.05680472821134E-06"
-        iyy="0.00293274601666501"
-        iyz="-4.85804534901831E-08"
-        izz="0.00503562271238706" />
-    </inertial>
-    <visual>
-      <origin
-        xyz="0 0 0"
-        rpy="0 0 0" />
-      <geometry>
-        <mesh
-          filename="file://$(find robot_description)/meshes/R5A_link2.STL" />
-      </geometry>
-      <material
-        name="">
-        <color
-          rgba="0.792156862745098 0.819607843137255 0.933333333333333 1" />
-      </material>
-    </visual>
-    <collision>
-      <origin
-        xyz="0 0 0"
-        rpy="0 0 0" />
-      <geometry>
-        <mesh
-          filename="file://$(find robot_description)/meshes/R5A_link2.STL" />
-      </geometry>
-    </collision>
-  </link>
-  <joint
-    name="R1_Pitch"
-    type="revolute">
-    <origin
-      xyz="-0.00310901547925538 0.1655 0"
-      rpy="0 0 0" />
-    <parent
-      link="R5A_link1" />
-    <child
-      link="R5A_link2" />
-    <axis
-      xyz="-0.999934112328875 0 -0.011479155067573" />
-    <limit
-      lower="-1.5"
-      upper="1.5"
-      effort="5"
-      velocity="1" />
-    <hardwareInterface>position</hardwareInterface>
-  </joint>
-  <link
-    name="R5A_link3">
-    <inertial>
-      <origin
-        xyz="-0.000315549279166789 0.042444959407996 0.00042316309562433"
-        rpy="0 0 0" />
-      <mass
-        value="0.749292336081855" />
-      <inertia
-        ixx="0.00200425601332893"
-        ixy="9.1795637501825E-06"
-        ixz="-2.55766332056785E-08"
-        iyy="0.000697358197450952"
-        iyz="-7.84063656624641E-06"
-        izz="0.00196480563389349" />
-    </inertial>
-    <visual>
-      <origin
-        xyz="0 0 0"
-        rpy="0 0 0" />
-      <geometry>
-        <mesh
-          filename="file://$(find robot_description)/meshes/R5A_link3.STL" />
-      </geometry>
-      <material
-        name="">
-        <color
-          rgba="0.792156862745098 0.819607843137255 0.933333333333333 1" />
-      </material>
-    </visual>
-    <collision>
-      <origin
-        xyz="0 0 0"
-        rpy="0 0 0" />
-      <geometry>
-        <mesh
-          filename="file://$(find robot_description)/meshes/R5A_link3.STL" />
-      </geometry>
-    </collision>
-  </link>
-  <joint
-    name="R2_Pitch"
-    type="revolute">
-    <origin
-      xyz="0.00300704230231069 0.221123792803564 0"
-      rpy="0 0 0" />
-    <parent
-      link="R5A_link2" />
-    <child
-      link="R5A_link3" />
-    <axis
-      xyz="-1 0 0" />
-    <limit
-      lower="-1.5"
-      upper="1.5"
-      effort="5"
-      velocity="1" />
-    <hardwareInterface>position</hardwareInterface>
-  </joint>
-  <link
-    name="R5A_link4">
-    <inertial>
-      <origin
-        xyz="-0.000206047771187218 0.0454873904143415 -0.000219105733632293"
-        rpy="0 0 0" />
-      <mass
-        value="0.355077243317478" />
-      <inertia
-        ixx="0.000669805200123062"
-        ixy="-4.71996739637697E-07"
-        ixz="-1.57736445584604E-07"
-        iyy="0.000358674558440891"
-        iyz="-5.41990968682589E-08"
-        izz="0.000768116251564114" />
-    </inertial>
-    <visual>
-      <origin
-        xyz="0 0 0"
-        rpy="0 0 0" />
-      <geometry>
-        <mesh
-          filename="file://$(find robot_description)/meshes/R5A_link4.STL" />
-      </geometry>
-      <material
-        name="">
-        <color
-          rgba="0.792156862745098 0.819607843137255 0.933333333333333 1" />
-      </material>
-    </visual>
-    <collision>
-      <origin
-        xyz="0 0 0"
-        rpy="0 0 0" />
-      <geometry>
-        <mesh
-          filename="file://$(find robot_description)/meshes/R5A_link4.STL" />
-      </geometry>
-    </collision>
-  </link>
-  <joint
-    name="R3_Yaw"
-    type="revolute">
-    <origin
-      xyz="0 0.1375 0"
-      rpy="0 0 0" />
-    <parent
-      link="R5A_link3" />
-    <child
-      link="R5A_link4" />
-    <axis
-      xyz="0 -0.999718303067734 -0.0237342476470231" />
-    <limit
-      lower="-1.5"
-      upper="1.5"
-      effort="5"
-      velocity="1" />
-    <hardwareInterface>position</hardwareInterface>
-  </joint>
-  <link
-    name="R5A_link5">
-    <inertial>
-      <origin
-        xyz="-0.000347552332670687 0.000167028378251888 0.0138173380766619"
-        rpy="0 0 0" />
-      <mass
-        value="0.198451767848984" />
-      <inertia
-        ixx="0.000113354976202718"
-        ixy="-9.1633661632938E-08"
-        ixz="2.54500165125599E-07"
-        iyy="8.47211726683811E-05"
-        iyz="4.4543875805716E-08"
-        izz="6.47134110451793E-05" />
-    </inertial>
-    <visual>
-      <origin
-        xyz="0 0 0"
-        rpy="0 0 0" />
-      <geometry>
-        <mesh
-          filename="file://$(find robot_description)/meshes/R5A_link5.STL" />
-      </geometry>
-      <material
-        name="">
-        <color
-          rgba="0.792156862745098 0.819607843137255 0.933333333333333 1" />
-      </material>
-    </visual>
-    <collision>
-      <origin
-        xyz="0 0 0"
-        rpy="0 0 0" />
-      <geometry>
-        <mesh
-          filename="file://$(find robot_description)/meshes/R5A_link5.STL" />
-      </geometry>
-    </collision>
-  </link>
-  <joint
-    name="R4_Pitch"
-    type="revolute">
-    <origin
-      xyz="0 0.0950000000000002 0"
-      rpy="1.5707963267949 0 3.14159265358979" />
-    <parent
-      link="R5A_link4" />
-    <child
-      link="R5A_link5" />
-    <axis
-      xyz="-0.995634790742834 0.0933346852058426 0" />
-    <limit
-      lower="-1.5"
-      upper="1.5"
-      effort="5"
-      velocity="1" />
-    <hardwareInterface>position</hardwareInterface>
-  </joint>
-  <link
-    name="R5A_GripperLeft_Link1">
-    <inertial>
-      <origin
-        xyz="-0.00659452357779758 -0.000394229793377554 2.33412007890428E-06"
-        rpy="0 0 0" />
-      <mass
-        value="0.00487858122952023" />
-      <inertia
-        ixx="2.28094324920978E-07"
-        ixy="1.69392169643129E-08"
-        ixz="-1.00081436396101E-10"
-        iyy="9.51062234425361E-07"
-        iyz="1.21242073786193E-09"
-        izz="1.15060635431209E-06" />
-    </inertial>
-    <visual>
-      <origin
-        xyz="0 0 0"
-        rpy="0 0 0" />
-      <geometry>
-        <mesh
-          filename="file://$(find robot_description)/meshes/R5A_GripperLeft_Link1.STL" />
-      </geometry>
-      <material
-        name="">
-        <color
-          rgba="1 1 1 1" />
-      </material>
-    </visual>
-    <collision>
-      <origin
-        xyz="0 0 0"
-        rpy="0 0 0" />
-      <geometry>
-        <mesh
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